Commit message: fix(urdf): correct base_footprint ground offset and wheel spacing
base_footprint_joint now offsets by -wheel_radius so it represents
true ground-contact height instead of floating at base_link's
height, fixing the robot appearing sunk below RViz's grid.

Adjusted wheel_offset_y to keep wheel separation consistent with
my_controllers.yaml's calibrated value.

File: description/robot_core.xacro (robot description, xacro)
@@ -5,10 +5,9 @@
     <xacro:property name="chassis_width" value="0.505"/>
     <xacro:property name="chassis_height" value="0.40"/>
-    <xacro:property name="chassis_mass" value="40.0"/>
     <xacro:property name="wheel_radius" value="0.1016"/>
     <xacro:property name="wheel_thickness" value="0.0508"/>
     <xacro:property name="wheel_mass" value="0.6"/>
     <xacro:property name="wheel_offset_x" value="0.265"/>
-    <xacro:property name="wheel_offset_y" value="0.1485"/>
+    <xacro:property name="wheel_offset_y" value="0.1625"/>
     <xacro:property name="wheel_offset_z" value="0.01"/>
     <xacro:property name="caster_wheel_radius" value="0.1016"/>
@@ -71,5 +70,5 @@
             </geometry>
         </collision>
-        <xacro:inertial_box mass="0.5" x="${chassis_length}" y="${chassis_width}" z="${chassis_height}">
+        <xacro:inertial_box mass="0.05" x="${chassis_length}" y="${chassis_width}" z="${chassis_height}">
             <origin xyz="${chassis_length/2} 0 ${chassis_height/2}" rpy="0 0 0"/>
         </xacro:inertial_box>
