Commit message: fix(urdf): remount camera on solar_mast instead of chassis
Camera joint now parents to solar_mast with a simple local offset
(0 0 0.135) instead of chassis with a large absolute offset and a
commented-out alternate origin. Mounting on the mast gives the
camera proper elevation for its field of view without needing to
hand-tune chassis-relative coordinates.

File: description/camera.xacro (robot description, xacro)
@@ -2,8 +2,7 @@
 <robot xmlns:xacro="http://www.ros.org/wiki/xacro" >
     <joint name="camera_joint" type="fixed">
-        <parent link="chassis"/>
+        <parent link="solar_mast"/>
         <child link="camera_link"/>
-       <!--<origin xyz="0.5 0 0.181" rpy="0 0.18 0"/>-->
-        <origin xyz="0.276 0 0.181" rpy="0 0.18 0"/>
+        <origin xyz="0 0 0.135"/>
     </joint>
     <link name="camera_link">
